File: hardware/carrier-hat/carrier-hat.kicad_pcb (KiCad board)
At the start: 2 copper layers, 65 x 30 mm, 4 parts

Commit message: ...
Parts:
- removed ? (x4): , MountingHole:MountingHole_2.7mm_M2.5
- added C1: 100nF, Resistor_SMD:R_0805_2012Metric, F.Cu at (20.0, 5.00)
- added D1: LED_3mm, LED_THT:LED_D3.0mm, F.Cu at (10.0, 26.0)
- added J1: PinHeader_2x20, Connector_PinHeader_2.54mm:PinHeader_2x20_P2.54mm_Vertical, F.Cu at (32.5, 15.0)
- added J2: JST_XH_8pin, Connector_JST:JST_XH_B8B-XH-A_1x08_P2.50mm_Horizontal, F.Cu at (58.0, 8.00)
- added J3: JST_XH_5pin, Connector_JST:JST_XH_B5B-XH-A_1x05_P2.50mm_Horizontal, F.Cu at (58.0, 20.0)
- added J4: JST_XH_2pin, Connector_JST:JST_XH_B2B-XH-A_1x02_P2.50mm_Horizontal, F.Cu at (10.0, 8.00)
- added MH1: MountingHole, MountingHole:MountingHole_2.7mm_M2.5, F.Cu at (3.50, 3.50)
- added MH2: MountingHole, MountingHole:MountingHole_2.7mm_M2.5, F.Cu at (61.5, 3.50)
- added MH3: MountingHole, MountingHole:MountingHole_2.7mm_M2.5, F.Cu at (3.50, 26.5)
- added MH4: MountingHole, MountingHole:MountingHole_2.7mm_M2.5, F.Cu at (61.5, 26.5)
- added R1: 220R, Resistor_SMD:R_0805_2012Metric, F.Cu at (10.0, 22.0)
Routing:
- net 3V3: track 0.00 -> 110.9 mm
- net GND: track 0.00 -> 88.3 mm, vias 0 -> 7
- net GPIO_INT: track 0.00 -> 43.0 mm
- net I2C1_SCL: track 0.00 -> 42.9 mm
- net I2C1_SDA: track 0.00 -> 42.8 mm
- net GPIO_LED: track 0.00 -> 32.5 mm
- net GPIO_RST: track 0.00 -> 31.4 mm
- net SPI0_CE0: track 0.00 -> 30.5 mm
- net SPI0_SCLK: track 0.00 -> 29.3 mm
- net GPIO_DC: track 0.00 -> 28.5 mm
- net SPI0_MOSI: track 0.00 -> 27.0 mm
- net GPIO_SHUTDOWN: track 0.00 -> 23.5 mm
- added copper zone on B.Cu, net GND
Other:
- board text added: "C1 100nF"
- board text added: "J4: SHUTDOWN"
